Commit message: Update project_robot.urdf

File: project_robot.urdf (robot description, URDF)
Before this commit: robot project_robot, 6 links, 5 joints
Links:
- added link base_footprint; visual box size=.01 .01 .01
Joints:
- added joint base_footprint_joint: type fixed, parent base_footprint, child basic_map, origin xyz=0 0 0 rpy=0 0 0
