Commit message: Update project_robot.urdf

File: project_robot/urdf/project_robot.urdf (robot description, URDF)
Before this commit: robot project_robot, 7 links, 6 joints
Links:
- added link LiDar; visual cylinder length=0.04 radius=0.05
- added link camera; visual cylinder length=.04 radius=0.02
- added link column1; visual cylinder length=.3 radius=0.01
- added link column2; visual cylinder length=.3 radius=0.01
- added link column3; visual cylinder length=.3 radius=0.01
- added link column4; visual cylinder length=.3 radius=0.01
- added link controller; visual box size=.2 .15 .03
- added link head2; visual box size=.1 .05 .05
- added link nozzle; visual box size=.14 .05 .02
- added link raspberry_pi; visual box size=.1 .2 .03
- added link sec_lev; visual cylinder length=0.04 radius=0.18
- added link top_lev; visual cylinder length=0.04 radius=0.18
- added link wire1; visual box size=.07 .1 .01
- added link wire2; visual box size=.02 .1 .01
- added link wirefromcon; visual box size=.07 .13 .01
- added link wirefromrasp; visual box size=.07 .13 .01
- added link wirefromwire; visual box size=.07 .15 .01
- link basic_map: geometry visual cylinder length=0.04 radius=0.18
- link head: geometry visual box size=.1 .05 .05
Joints:
- removed joint tobox
- added joint camhead: type fixed, parent basic_map, child head, origin xyz=0 0.1 0.05
- added joint conto: type fixed, parent controller, child wirefromcon, origin xyz=0 -0.1 0.005
- added joint contocam: type fixed, parent controller, child wire1, origin xyz=0 0.1 0.005
- added joint nozhead: type fixed, parent sec_lev, child head2, origin xyz=0 0.1 0.05
- added joint raspto: type fixed, parent raspberry_pi, child wirefromrasp, origin xyz=0 -0.1 0
- added joint rasptonoz: type fixed, parent raspberry_pi, child wire2, origin xyz=0 0.1 0.005 rpy=0 0 0
- added joint toLia: type fixed, parent top_lev, child LiDar, origin xyz=0 0.1 .02 rpy=0 0 0
- added joint tocamera: type fixed, parent head, child camera, origin xyz=0 0.03 0 rpy=1.57075 0 0
- added joint tocol1: type fixed, parent basic_map, child column1, origin xyz=0.12 0.12 0.15 rpy=0 0 0
- added joint tocol2: type fixed, parent basic_map, child column2, origin xyz=-0.12 0.12 0.15 rpy=0 0 0
- added joint tocol3: type fixed, parent basic_map, child column3, origin xyz=0.12 -0.12 0.15 rpy=0 0 0
- added joint tocol4: type fixed, parent basic_map, child column4, origin xyz=-0.12 -0.12 0.15 rpy=0 0 0
- added joint tocon: type fixed, parent basic_map, child controller, origin xyz=0 -0.04 0.03
- added joint tolev2: type fixed, parent basic_map, child sec_lev, origin xyz=0 0 0.15 rpy=0 0 0
- added joint tonoz: type fixed, parent head2, child nozzle, origin xyz=0 0.03 0
- added joint torasp: type fixed, parent sec_lev, child raspberry_pi, origin xyz=0 -0.04 0.03
- added joint totop: type fixed, parent basic_map, child top_lev, origin xyz=0 0 0.3 rpy=0 0 0
- added joint wireto: type fixed, parent wirefromcon, child wirefromwire, origin xyz=0 -0.06 0.07 rpy=1.55 0 0
- joint base_footprint_joint: origin xyz=0 0 0 rpy=0 0 0 -> xyz=0 0 0 rpy=0 0 5
- joint left_back_wheel_joint: origin xyz=-0.08 -0.2 -0.03 rpy=0 1.57075 0 -> xyz=-0.08 -0.1 -0.03 rpy=0 1.57075 0
- joint left_front_wheel_joint: origin xyz=-0.08 0.2 -0.03 rpy=0 1.57075 0 -> xyz=-0.08 0.1 -0.03 rpy=0 1.57075 0
- joint right_back_wheel_joint: origin xyz=0.08 -0.2 -0.03 rpy=0 1.57075 0 -> xyz=0.08 -0.1 -0.03 rpy=0 1.57075 0
- joint right_front_wheel_joint: origin xyz=0.08 0.2 -0.03 rpy=0 1.57075 0 -> xyz=0.08 0.1 -0.03 rpy=0 1.57075 0
